Commit message: add a camera and a 3D lidar

File: track_master_project/track_master/urdf/chassis.xacro (robot description, xacro)
@@ -3,4 +3,5 @@
   <!-- Include the parameters file -->
   <xacro:include filename="$(find track_master)/urdf/robot_parameters.xacro" />
+  <xacro:include filename="$(find track_master)/urdf/inertial_macros.xacro"/>
   <!-- Couleurs -->
   <material name="white">
@@ -25,9 +26,7 @@
       </geometry>
     </collision>
-    <inertial>
-      <mass value="2.0"/>
-      <origin xyz="0 0 0"/>
-      <inertia ixx="0.1" ixy="0.0" ixz="0.0" iyy="0.1" iyz="0.0" izz="0.1"/>
-    </inertial>
+    <xacro:inertial_box mass="0.5" x="${chassis_length}" y="${chassis_width}" z="${chassis_height}">
+            <origin xyz="${chassis_length/2} 0 ${chassis_height/2}" rpy="0 0 0"/>
+    </xacro:inertial_box>
   </link>
   <!-- Gazebo plugin for base link -->
@@ -39,5 +38,5 @@
     <parent link="base_footprint"/>
     <child link="base_link"/>
-    <origin xyz="0 0 0.15" rpy="0 0 0"/>
+    <origin xyz="0 0 0.075" rpy="0 0 0"/>
   </joint>
   <!-- Rear left wheel -->
@@ -54,16 +53,14 @@
       </geometry>
     </collision>
-    <inertial>
-      <mass value="0.3"/>
-      <origin xyz="0 0 0"/>
-      <inertia ixx="0.01" ixy="0.0" ixz="0.0" iyy="0.01" iyz="0.0" izz="0.01"/>
-    </inertial>
+    <xacro:inertial_cylinder mass="0.3" length="${rear_wheel_length}" radius="${rear_wheel_radius}">
+            <origin xyz="0 0 0" rpy="0 0 0"/>
+    </xacro:inertial_cylinder>
   </link>
   <gazebo reference="rear_left_wheel">
     <material>Gazebo/Blue</material>
-    <!--<mu1>0.9</mu1>
+    <mu1>0.9</mu1>
     <mu2>0.9</mu2>
     <kp>1000000.0</kp>
-    <kd>1.0</kd>-->
+    <kd>1.0</kd>
   </gazebo>
   <!-- Rear right wheel -->
@@ -80,12 +77,14 @@
       </geometry>
     </collision>
-    <inertial>
-      <mass value="0.3"/>
-      <origin xyz="0 0 0"/>
-      <inertia ixx="0.01" ixy="0.0" ixz="0.0" iyy="0.01" iyz="0.0" izz="0.01"/>
-    </inertial>
+    <xacro:inertial_cylinder mass="0.3" length="${rear_wheel_length}" radius="${rear_wheel_radius}">
+            <origin xyz="0 0 0" rpy="0 0 0"/>
+    </xacro:inertial_cylinder>
   </link>
   <gazebo reference="rear_right_wheel">
     <material>Gazebo/Blue</material>
+    <mu1>0.9</mu1>
+    <mu2>0.9</mu2>
+    <kp>1000000.0</kp>
+    <kd>1.0</kd>
   </gazebo>
   <!-- Front left wheel -->
@@ -102,12 +101,14 @@
       </geometry>
     </collision>
-    <inertial>
-      <mass value="0.3"/>
-      <origin xyz="0 0 0"/>
-      <inertia ixx="0.01" ixy="0.0" ixz="0.0" iyy="0.01" iyz="0.0" izz="0.01"/>
-    </inertial>
+    <xacro:inertial_cylinder mass="0.3" length="${front_wheel_length}" radius="${front_wheel_radius}">
+            <origin xyz="0 0 0" rpy="0 0 0"/>
+    </xacro:inertial_cylinder>
   </link>
   <gazebo reference="front_left_wheel">
     <material>Gazebo/Blue</material>
+    <mu1>0.9</mu1>
+    <mu2>0.9</mu2>
+    <kp>1000000.0</kp>
+    <kd>1.0</kd>
   </gazebo>
   <!-- Front right wheel -->
@@ -124,12 +125,14 @@
       </geometry>
     </collision>
-    <inertial>
-      <mass value="0.3"/>
-      <origin xyz="0 0 0"/>
-      <inertia ixx="0.01" ixy="0.0" ixz="0.0" iyy="0.01" iyz="0.0" izz="0.01"/>
-    </inertial>
+    <xacro:inertial_cylinder mass="0.3" length="${front_wheel_length}" radius="${front_wheel_radius}">
+            <origin xyz="0 0 0" rpy="0 0 0"/>
+    </xacro:inertial_cylinder>
   </link>
   <gazebo reference="front_right_wheel">
     <material>Gazebo/Blue</material>
+    <mu1>0.9</mu1>
+    <mu2>0.9</mu2>
+    <kp>1000000.0</kp>
+    <kd>1.0</kd>
   </gazebo>
   <!-- Joints for each wheel -->
@@ -139,4 +142,6 @@
     <origin xyz="${rear_left_wheel_pos_x} ${rear_left_wheel_pos_y} 0" rpy="-${pi/2}  0 0"/>
     <axis xyz="0 0 1"/>
+    <limit effort="10.0" velocity="9.0"/>
+    <dynamics damping="0.01" friction="0.05"/>
   </joint>
   <joint name="rear_right_wheel_joint" type="continuous">
@@ -145,4 +150,6 @@
     <origin xyz="${rear_right_wheel_pos_x} ${rear_right_wheel_pos_y} 0" rpy="-${pi/2}   0 0"/>
     <axis xyz="0 0 1"/>
+    <limit effort="10.0" velocity="9.0"/>
+    <dynamics damping="0.01" friction="0.05"/>
   </joint>
   <joint name="front_left_wheel_joint" type="continuous">
@@ -151,4 +158,6 @@
     <origin xyz="${front_left_wheel_pos_x} ${front_left_wheel_pos_y} 0" rpy="-${pi/2}   0 0"/>
     <axis xyz="0 0 1"/>
+    <limit effort="10.0" velocity="9.0"/>
+    <dynamics damping="0.01" friction="0.05"/>
   </joint>
   <joint name="front_right_wheel_joint" type="continuous">
@@ -157,4 +166,6 @@
     <origin xyz="${front_right_wheel_pos_x} ${front_right_wheel_pos_y} 0" rpy="-${pi/2} 0 0"/>
     <axis xyz="0 0 1"/>
+    <limit effort="10.0" velocity="9.0"/>
+    <dynamics damping="0.01" friction="0.05"/>
   </joint>
 </robot>

File: track_master_project/track_master/urdf/robot_parameters.xacro (robot description, xacro)
@@ -19,7 +19,4 @@
   <xacro:property name="front_left_wheel_pos_y" value="0.18"/>
   <xacro:property name="front_right_wheel_pos_y" value="-0.18"/>
-  <!-- Parameters for steering limits -->
-  <xacro:property name="steering_limit_lower" value="-0.785"/>
-  <xacro:property name="steering_limit_upper" value="0.785"/>
   <!-- Parameters for sensor positions -->
   <xacro:property name="gps_pos_x" value="0.05"/>

File: track_master_project/track_master/urdf/ros2_control.xacro (robot description, xacro)
@@ -7,6 +7,6 @@
         <joint name="front_right_wheel_joint">
             <command_interface name="velocity">
-                <param name="min">-5</param> <!--expressed in rad/s-->
-                <param name="max">5</param>
+                <param name="min">-9</param> <!--expressed in rad/s-->
+                <param name="max">9</param>
             </command_interface>
             <state_interface name="velocity"></state_interface>
@@ -15,6 +15,6 @@
         <joint name="front_left_wheel_joint">
             <command_interface name="velocity">
-                <param name="min">-5</param>
-                <param name="max">5</param>
+                <param name="min">-9</param> <!--expressed in rad/s-->
+                <param name="max">9</param>
             </command_interface>
             <state_interface name="velocity"></state_interface>
@@ -23,6 +23,6 @@
         <joint name="rear_right_wheel_joint">
             <command_interface name="velocity">
-                <param name="min">-5</param>
-                <param name="max">5</param>
+                <param name="min">-9</param> <!--expressed in rad/s-->
+                <param name="max">9</param>
             </command_interface>
             <state_interface name="velocity"></state_interface>
@@ -31,6 +31,6 @@
         <joint name="rear_left_wheel_joint">
             <command_interface name="velocity">
-                <param name="min">-5</param>
-                <param name="max">5</param>
+                <param name="min">-9</param> <!--expressed in rad/s-->
+                <param name="max">9</param>
             </command_interface>
             <state_interface name="velocity"></state_interface>

File: track_master_project/track_master/urdf/tracker_master_bot.urdf.xacro (robot description, xacro)
@@ -2,5 +2,5 @@
 <robot xmlns:xacro="http://www.ros.org/wiki/xacro" name="tracker_master_bot">
   <!-- Include the parameter file -->
-  <!--<xacro:include filename="$(find track_master)/urdf/robot_parameters.xacro" / -->
+  <xacro:include filename="$(find track_master)/urdf/robot_parameters.xacro" />
   <!-- Include the chassis -->
   <xacro:include filename="$(find track_master)/urdf/chassis.xacro" />
@@ -9,4 +9,7 @@
   <!-- Include the IMU sensor -->
   <xacro:include filename="$(find track_master)/urdf/imu_sensor.xacro" />
+ <!-- <xacro:include filename="$(find track_master)/urdf/lidar.xacro" /> -->
+   <xacro:include filename="$(find track_master)/urdf/point_cloud_lidar.xacro" />
+  <xacro:include filename="$(find track_master)/urdf/camera.xacro" />
   <xacro:include filename="$(find track_master)/urdf/ros2_control.xacro" />
 </robot>
