Commit message: update robot urdf

File: src/track_master/urdf/imu_sensor.xacro (robot description, xacro)
@@ -11,5 +11,5 @@
     <parent link="base_link"/>
     <child link="imu_link"/>
-    <origin xyz="${imu_pos_x} ${imu_pos_y} ${imu_pos_z}"/>
+    <origin xyz="${imu_pos_x} ${imu_pos_y} ${imu_pos_z}" rpy="0 0 0"/>
   </joint>
   <link name="imu_link">
@@ -19,5 +19,5 @@
       </geometry>
     </visual>
-    <origin xyz="${imu_pos_x} ${imu_pos_y} ${imu_pos_z}"/>
+    <origin xyz="${imu_pos_x} ${imu_pos_y} ${imu_pos_z}" rpy="0 0 0"/>
   </link>
   <!-- IMU sensor in Gazebo -->
@@ -26,20 +26,59 @@
       Gazebo/Vert
     </material>
-    <gravity>true</gravity>
+    <gravity>false</gravity>
     <sensor name="imu_sensor" type="imu">
       <always_on>true</always_on>
-      <update_rate>10</update_rate>
+      <update_rate>10</update_rate> <!-- Augmenté pour plus de précision -->
       <visualize>true</visualize>
       <topic>/imu/data</topic>
+      <!-- Configuration de l'IMU avec du bruit -->
+      <imu>
+        <angular_velocity>
+          <x>
+            <noise type="gaussian">
+              <mean>0.0</mean>
+              <stddev>0.01</stddev>
+            </noise>
+          </x>
+          <y>
+            <noise type="gaussian">
+              <mean>0.0</mean>
+              <stddev>0.01</stddev>
+            </noise>
+          </y>
+          <z>
+            <noise type="gaussian">
+              <mean>0.0</mean>
+              <stddev>0.01</stddev>
+            </noise>
+          </z>
+        </angular_velocity>
+        <linear_acceleration>
+          <x>
+            <noise type="gaussian">
+              <mean>0.0</mean>
+              <stddev>0.02</stddev>
+            </noise>
+          </x>
+          <y>
+            <noise type="gaussian">
+              <mean>0.0</mean>
+              <stddev>0.02</stddev>
+            </noise>
+          </y>
+          <z>
+            <noise type="gaussian">
+              <mean>0.0</mean>
+              <stddev>0.02</stddev>
+            </noise>
+          </z>
+        </linear_acceleration>
+      </imu>
+      <!-- Plugin IMU Gazebo -->
       <plugin filename="libgazebo_ros_imu_sensor.so" name="imu_plugin">
         <ros>
           <remapping>~/out:=/imu/data</remapping>
         </ros>
-        <bodyName>imu_link</bodyName>
-        <updateRateHZ>10.0</updateRateHZ>
-        <gaussianNoise>0.01</gaussianNoise>
-        <xyzOffset>0 0 0</xyzOffset>
-        <rpyOffset>0 0 0</rpyOffset>
-        <frameName>imu_link</frameName>
+        <frame_name>imu_link</frame_name>
         <initial_orientation_as_reference>false</initial_orientation_as_reference>
       </plugin>

File: src/track_master/urdf/ros2_control.xacro (robot description, xacro)
@@ -7,6 +7,6 @@
         <joint name="front_right_wheel_joint">
             <command_interface name="velocity">
-                <param name="min">-9</param> <!--expressed in rad/s-->
-                <param name="max">9</param>
+                <param name="min">-20</param> <!--expressed in rad/s-->
+                <param name="max">20</param>
             </command_interface>
             <state_interface name="velocity"></state_interface>
@@ -15,6 +15,6 @@
         <joint name="front_left_wheel_joint">
             <command_interface name="velocity">
-                <param name="min">-9</param> <!--expressed in rad/s-->
-                <param name="max">9</param>
+                <param name="min">-20</param> <!--expressed in rad/s-->
+                <param name="max">20</param>
             </command_interface>
             <state_interface name="velocity"></state_interface>
@@ -23,6 +23,6 @@
         <joint name="rear_right_wheel_joint">
             <command_interface name="velocity">
-                <param name="min">-9</param> <!--expressed in rad/s-->
-                <param name="max">9</param>
+                <param name="min">-20</param> <!--expressed in rad/s-->
+                <param name="max">20</param>
             </command_interface>
             <state_interface name="velocity"></state_interface>
@@ -31,6 +31,6 @@
         <joint name="rear_left_wheel_joint">
             <command_interface name="velocity">
-                <param name="min">-9</param> <!--expressed in rad/s-->
-                <param name="max">9</param>
+                <param name="min">-20</param> <!--expressed in rad/s-->
+                <param name="max">20</param>
             </command_interface>
             <state_interface name="velocity"></state_interface>
@@ -41,5 +41,5 @@
         <plugin name="gazebo_ros2_control" filename="libgazebo_ros2_control.so">
             <parameters>
-                $(find robot_control)/config/diff_drive_controller.yaml
+                $(find track_master_control)/config/diff_drive_controller.yaml
             </parameters>
         </plugin>
